File: hardware/pcb/material_weight_calculator.kicad_pcb (KiCad board)
At the start: 2 copper layers, 82 x 68 mm, 20 parts, among them J1 KEYPAD_8PIN, J2 BATTERY_3AAA, J3 SHARP_3502_CABLE, J4 UPDI_3V3, Q1 2N3906, U1 AVR128DA28-I/SP, U2 MCP1700-3302E/TO

Commit message: Revise calculator for 2.8-inch UC1701 display with adapter PCB and larger resin bezel
Replace the Sharp display with ERC12864FS-655. Regenerate CAD, STLs, schematics, routed PCBs, Gerbers, drills, print templates and R2 download packages. Preserve the 4x4 keypad and AAA supply. Verify both PCB DRC reports, manufacturer pin map, closed meshes, nominal fit and package checksums. Physical testing and device firmware remain pending.
Parts:
- J3: value SHARP_3502_CABLE -> UC1701_ADAPTER_CABLE; footprint MW_footprints:PinHeader_1x09_P2.54mm_Vertical -> MW_footprints:PinHeader_1x08_P2.54mm_Vertical
- Q1: value 2N3906 -> onsemi 2N3906 EBC
Connections:
- J3 pad 2: (no net) -> GND
- J3 pad 3: GND -> LCD_CLK
- J3 pad 4: LCD_CLK -> LCD_DATA
- J3 pad 5: LCD_DATA -> LCD_CS
- J3 pad 6: LCD_CS -> LCD_CD
- J3 pad 7: GND -> LCD_RST
- J3 pad 8: LCD_DISP -> (no net)
- U1 pad 26: LCD_DISP -> LCD_CD
- U1 pad 27: (no net) -> LCD_RST
Routing:
- net LCD_CD: track 0.00 -> 56.6 mm
- net LCD_RST: track 0.00 -> 46.9 mm, vias 0 -> 3
- net LCD_DISP: track 36.3 -> 0.00 mm, vias 3 -> 0
- net LCD_CS: track 49.5 -> 46.9 mm
- net LCD_CLK: track 36.8 -> 39.3 mm
- net LCD_DATA: track 31.7 -> 34.2 mm
- net GND: track 179.5 -> 177.9 mm
Other:
- board text added: "J3: UC1701 8-WIRE"
- board text added: "MATERIAL WEIGHT R2"
- board text removed: "J3 PIN 2: NO WIRE"
- board text removed: "MATERIAL WEIGHT R1"
