File: hardware/pcb/material_weight_calculator.kicad_sch (KiCad schematic)
At the start: 16 parts, among them J1 KEYPAD_8PIN, J2 BATTERY_3AAA, J3 SHARP_3502_CABLE, J4 UPDI_3V3, Q1 2N3906, U1 AVR128DA28-I/SP, U2 MCP1700-3302E/TO

Commit message: Revise calculator for 2.8-inch UC1701 display with adapter PCB and larger resin bezel
Replace the Sharp display with ERC12864FS-655. Regenerate CAD, STLs, schematics, routed PCBs, Gerbers, drills, print templates and R2 download packages. Preserve the 4x4 keypad and AAA supply. Verify both PCB DRC reports, manufacturer pin map, closed meshes, nominal fit and package checksums. Physical testing and device firmware remain pending.
Parts:
- J3: value SHARP_3502_CABLE -> UC1701_ADAPTER_CABLE; footprint MW_footprints:PinHeader_1x09_P2.54mm_Vertical -> MW_footprints:PinHeader_1x08_P2.54mm_Vertical
- Q1: value 2N3906 -> onsemi 2N3906 EBC
Connections:
- net GND: now also J3.2 (GND); no longer J3.3 (GND), J3.7 (EXTMODE), J3.9 (EXTCOMIN)
- net LCD_CLK: now also J3.3 (SCK); no longer J3.4 (CLK)
- net LCD_CS: now also J3.5 (CS_N); no longer J3.6 (CS)
- net LCD_DATA: now also J3.4 (SDA); no longer J3.5 (DI)
- net LCD_RST: now reaches U1.27 (PA5)
- net LCD_RST: now also J3.7 (RST_N)
- net LCD_DISP: no longer names the net of J3.8 (NC)
- net LCD_DISP: no longer U1.26 (PA4)
- new net LCD_CD: J3.6 (CD), U1.26 (PA4)
- no-connect marks 11 -> 10
